File: Oscilloscope_Differential_Probe/KiCAD/Diff_probe.sch (KiCad schematic (older format))
At the start: 33 parts, among them J1 Conn_01x02, J1.1 Conn_Coaxial, J1.2 Conn_Coaxial, J2 Conn_Coaxial, J3 Conn_01x01_Female, J4 Conn_01x01_Female, SW1 SPST, U1 LTC6268-10, U2 LTC6268-10, U3 LT1761-5

Commit message: BOM generated
Parts:
- J1: MouserID (none) -> TSW-104-12-T-S-RA
- U1, U2: MouserID (none) -> 584-C6268IS6-10TMPF
- U3: MouserID (none) -> 584-LT1761ES5-5TRPBF
Changed lines of the file:
@@
 F 2 "Connector_PinHeader_2.54mm:PinHeader_1x02_P2.54mm_Vertical" H 3300 4100 50  0001 C CNN
 F 3 "~" H 3300 4100 50  0001 C CNN
+F 4 "TSW-104-12-T-S-RA" H 3300 4100 50  0001 C CNN "MouserID"
 	1    3300 4100
 	-1   0    0    1
@@
 F 2 "Package_TO_SOT_SMD:SOT-23-6" H 5850 4250 50  0001 C CNN
 F 3 "https://www.analog.com/media/en/technical-documentation/data-sheets/OP07.pdf" H 5850 4350 50  0001 C CNN
+F 4 "584-C6268IS6-10TMPF" H 5800 4200 50  0001 C CNN "MouserID"
 	1    5800 4200
 	1    0    0    -1
@@
 F 2 "Package_TO_SOT_SMD:TSOT-23-5" H 5750 3375 50  0001 C CNN
 F 3 "https://www.analog.com/media/en/technical-documentation/data-sheets/1761sff.pdf" H 5750 3050 50  0001 C CNN
+F 4 "584-LT1761ES5-5TRPBF" H 5750 3050 50  0001 C CNN "MouserID"
 	1    5750 3050
 	1    0    0    -1
@@
 F 2 "Package_TO_SOT_SMD:SOT-23-6" H 7600 4250 50  0001 C CNN
 F 3 "https://www.analog.com/media/en/technical-documentation/data-sheets/OP07.pdf" H 7600 4350 50  0001 C CNN
+F 4 "584-C6268IS6-10TMPF" H 7550 4200 50  0001 C CNN "MouserID"
 	1    7550 4200
 	1    0    0    -1

Commit message: BOM updated
Parts:
- C1, C2: Vendor (none) -> Mouser; Vendor_No (none) -> 80-C1210C222JDGAUTO
- C3, C4, C5, C8, C9: Vendor (none) -> Mouser; Vendor_No (none) -> 80-C0805C103J5GECLR
- C6, C7: Vendor (none) -> Mouser; Vendor_No (none) -> 80-C0805C105K4R
- D1: Vendor (none) -> Mouser; Vendor_No (none) -> 604-APT3216LSECKJ4RV
- J1: Vendor (none) -> Mouser; Vendor_No (none) -> TSW-104-12-T-S-RA
- J1.1, J1.2, J2: Vendor (none) -> Mouser; Vendor_No (none) -> 223-CON-SMA-EDGE-S
- J3: Vendor (none) -> Mouser; Vendor_No (none) -> 534-593
- J4: Vendor (none) -> Mouser; Vendor_No (none) -> 534-594
- R1, R2: Vendor (none) -> Mouser; Vendor_No (none) -> 284-APC0805B49K9N
- R10: Vendor (none) -> Mouser; Vendor_No (none) -> 284-APC0805B499RN
- R11: Vendor (none) -> Mouser; Vendor_No (none) -> 667-ERA-6AEB54R9V
- R12: Vendor (none) -> Mouser; Vendor_No (none) -> 667-ERA-6AEB48R7V
- R13: Vendor (none) -> Mouser; Vendor_No (none) -> 71-CRCW120675R0FKEAC
- R3, R5: Vendor (none) -> Mouser; Vendor_No (none) -> 667-ERA-6AEB5490V
- R4, R7, R8: Vendor (none) -> Mouser; Vendor_No (none) -> 284-APC0805B10K0N
- R6: Vendor (none) -> Mouser; Vendor_No (none) -> 284-APC0805B4K99N
- R9: Vendor (none) -> Mouser; Vendor_No (none) -> 667-ERA-6AEB1913V
- SW1: Vendor (none) -> Mouser; Vendor_No (none) -> 642-DM01
- U1, U2: Vendor (none) -> Mouser; Vendor_No (none) -> 584-C6268IS6-10TMPF
- U3: Vendor (none) -> Mouser; Vendor_No (none) -> 584-LT1761ES5-5TRPBF

Commit message: update
Parts:
- C1, C2: In basket (none) -> Yes
Changed lines of the file:
@@
 F 5 "Mouser" H 4150 4000 50  0001 C CNN "Vendor"
 F 6 "80-C1210C222JDGAUTO" H 4150 4000 50  0001 C CNN "Vendor_No"
+F 7 "Yes" H 4150 4000 50  0001 C CNN "In basket"
 	1    4150 4000
 	0    1    1    0
@@
 F 5 "Mouser" H 4150 4400 50  0001 C CNN "Vendor"
 F 6 "80-C1210C222JDGAUTO" H 4150 4400 50  0001 C CNN "Vendor_No"
+F 7 "Yes" H 4150 4400 50  0001 C CNN "In basket"
 	1    4150 4400
 	0    1    1    0
